Commit message: Reallyuseful robot

File: description/camera.xacro (robot description, xacro)
@@ -2,31 +2,36 @@
 <robot xmlns:xacro="http://www.ros.org/wiki/xacro" >
     <joint name="camera_joint" type="fixed">
-        <parent link="chassis"/>
+        <origin rpy="0 0 0" xyz="0.07175 -0.072 0.33"/>
+        <parent link="head"/>
         <child link="camera_link"/>
-        <origin xyz="0.276 0 0.181" rpy="0 0.18 0"/>
-    </joint>
+      </joint>
     <link name="camera_link">
+        <inertial>
+            <origin rpy="0 0 0" xyz="-0.001604468363459316 0.07205272744017827 -0.002548711859325259"/>
+            <mass value="0.3739643327489875"/>
+            <inertia ixx="0.001081" ixy="0.0" ixz="1e-06" iyy="0.000322" iyz="0.0" izz="0.001051"/>
+        </inertial>
         <visual>
+            <origin rpy="0 0 0" xyz="-0.18275 0.072 -1.335"/>
             <geometry>
-                <box size="0.010 0.03 0.03"/>
+            <mesh filename="file://$(find articubot_one)/meshes/camera_link.stl" scale="0.001 0.001 0.001"/>
             </geometry>
-            <material name="black"/>
+            <material name="white"/>
         </visual>
-        <visual>
-            <origin xyz="0 0 -0.05"/>
+        <collision>
+            <origin rpy="0 0 0" xyz="-0.18275 0.072 -1.335"/>
             <geometry>
-                <cylinder radius="0.002" length="0.1"/>
+            <mesh filename="file://$(find articubot_one)/meshes/camera_link.stl" scale="0.001 0.001 0.001"/>
             </geometry>
-            <material name="black"/>
-        </visual>
+        </collision>
     </link>
     <joint name="camera_optical_joint" type="fixed">
         <parent link="camera_link"/>
         <child link="camera_link_optical"/>
-        <origin xyz="0 0 0" rpy="${-pi/2} 0 ${-pi/2}"/>
+        <origin xyz="0 0 0" rpy="1.5701 0 1.5701"/>
     </joint>
     <link name="camera_link_optical"></link>
     <gazebo reference="camera_link">
-        <material>Gazebo/Black</material>
+        <material>Gazebo/White</material>
         <sensor name="camera" type="camera">
             <pose> 0 0 0 0 0 0 </pose>

File: description/gazebo_control.xacro (robot description, xacro)
@@ -4,8 +4,8 @@
         <plugin name="diff_drive" filename="libgazebo_ros_diff_drive.so">
             <!-- Wheel Information -->
-            <left_joint>left_wheel_joint</left_joint>
-            <right_joint>right_wheel_joint</right_joint>
-            <wheel_separation>0.297</wheel_separation>
-            <wheel_diameter>0.066</wheel_diameter>
+            <left_joint>motor_left</left_joint>
+            <right_joint>motor_right</right_joint>
+            <wheel_separation>0.36</wheel_separation>
+            <wheel_diameter>0.20</wheel_diameter>
             <!-- Limits -->
             <max_wheel_torque>200</max_wheel_torque>

File: description/lidar.xacro (robot description, xacro)
@@ -1,59 +1,67 @@
 <?xml version="1.0"?>
 <robot xmlns:xacro="http://www.ros.org/wiki/xacro" >
-    <joint name="laser_joint" type="fixed">
-        <parent link="chassis"/>
-        <child link="laser_frame"/>
-        <origin xyz="0.122 0 0.212" rpy="0 0 0"/>
-    </joint>
-    <link name="laser_frame">
+    <joint name="Rigid8" type="fixed">
+        <origin rpy="0 0 0" xyz="-0.0675 -0.0002 0.05"/>
+        <parent link="lid"/>
+        <child link="lidar"/>
+      </joint>
+    <link name="lidar">
+        <inertial>
+            <origin rpy="0 0 0" xyz="-2.3483549826952554e-09 -3.4770506128023716e-07 0.009561590682608923"/>
+            <mass value="0.0886181648250366"/>
+            <inertia ixx="3.3e-05" ixy="0.0" ixz="0.0" iyy="3.3e-05" iyz="0.0" izz="6e-05"/>
+        </inertial>
         <visual>
+            <origin rpy="0 0 0" xyz="-0.1575 0.0 -0.3"/>
             <geometry>
-                <cylinder radius="0.05" length="0.04"/>
-            </geometry>
-            <material name="black"/>
-        </visual>
-        <visual>
-            <origin xyz="0 0 -0.05"/>
-            <geometry>
-                <cylinder radius="0.01" length="0.1"/>
+            <mesh filename="file://$(find articubot_one)/meshes/lidar.stl" scale="0.001 0.001 0.001"/>
             </geometry>
             <material name="black"/>
         </visual>
         <collision>
+            <origin rpy="0 0 0" xyz="-0.1575 0.0 -0.3"/>
             <geometry>
-                <cylinder radius="0.05" length="0.04"/>
+            <mesh filename="file://$(find articubot_one)/meshes/lidar.stl" scale="0.001 0.001 0.001"/>
             </geometry>
         </collision>
-        <xacro:inertial_cylinder mass="0.1" length="0.04" radius="0.05">
-            <origin xyz="0 0 0" rpy="0 0 0"/>
-        </xacro:inertial_cylinder>
     </link>
-    <gazebo reference="laser_frame">
+    <gazebo reference="lidar">
         <material>Gazebo/Black</material>
-        <sensor name="laser" type="ray">
-            <pose> 0 0 0 0 0 0 </pose>
-            <visualize>false</visualize>
-            <update_rate>10</update_rate>
-            <ray>
-                <scan>
-                    <horizontal>
-                        <samples>360</samples>
-                        <min_angle>-3.14</min_angle>
-                        <max_angle>3.14</max_angle>
-                    </horizontal>
-                </scan>
-                <range>
-                    <min>0.3</min>
-                    <max>12</max>
-                </range>
-            </ray>
-            <plugin name="laser_controller" filename="libgazebo_ros_ray_sensor.so">
-                <ros>
-                    <argument>~/out:=scan</argument>
-                </ros>
-                <output_type>sensor_msgs/LaserScan</output_type>
-                <frame_name>laser_frame</frame_name>
-            </plugin>
+        <sensor type="ray" name="ray">
+          <pose>0 0 0 0 0 0</pose>
+          <visualize>false</visualize>
+          <update_rate>10</update_rate>
+          <ray>
+            <scan>
+              <horizontal>
+                <samples>720</samples>
+                <resolution>1</resolution>
+                <min_angle>-2.87979</min_angle>
+                <max_angle>2.87979</max_angle>
+              </horizontal>
+            </scan>
+            <range>
+              <min>0.10</min>
+              <max>20.0</max>
+              <resolution>0.01</resolution>
+            </range>
+            <noise>
+              <type>gaussian</type>
+              <!-- Noise parameters based on published spec for Hokuyo laser
+                   achieving "+-30mm" accuracy at range < 10m.  A mean of 0.0m and
+                   stddev of 0.01m will put 99.7% of samples within 0.03m of the true
+                   reading. -->
+              <mean>0.0</mean>
+              <stddev>0.01</stddev>
+            </noise>
+          </ray>
+          <plugin name="laser_controller" filename="libgazebo_ros_ray_sensor.so">
+            <ros>
+                <argument>--ros-args --remap ~/out:=scan</argument>
+            </ros>
+            <output_type>sensor_msgs/LaserScan</output_type>
+            <frameName>lidar</frameName>
+          </plugin>
         </sensor>
-    </gazebo>
+      </gazebo>
 </robot>
